File: 2022-SHIELD-Arduino-FlexSensor/2022-SHIELD-Arduino-FlexSensor.kicad_pcb (KiCad board)
At the start: 2 copper layers, 68.6 x 53.3 mm, 12 parts, among them P1 Power, P2 Analog, P3 Digital, P4 Digital, P5 CONN_01X01, P6 CONN_01X01, P7 CONN_01X01, P8 CONN_01X01

Commit message: Add files via upload
Parts:
- removed REF**: HC-05, SHIELD_print_Library:HC-05
- removed REF**: OLED_0.91, SHIELD_print_Library:SIP-4
- removed REF**: KY-040, SHIELD_print_Library:KY-040
- removed REF**: LTC1050, SHIELD_print_Library:LTC1050
- added C1: 100n, Capacitor_THT:C_Disc_D4.3mm_W1.9mm_P5.00mm, F.Cu at (135.1, 111.2)
- added C2: 100n, Capacitor_THT:C_Disc_D7.5mm_W5.0mm_P7.50mm, F.Cu at (154.7, 105.9)
- added C3: 100n, Capacitor_THT:C_Disc_D4.3mm_W1.9mm_P5.00mm, F.Cu at (116.5, 97.4)
- added C4: 1u, Capacitor_THT:C_Rect_L7.0mm_W4.5mm_P5.00mm, F.Cu at (142.5, 100.9)
- added R0: Rsensor, Resistor_THT:R_Axial_DIN0207_L6.3mm_D2.5mm_P7.62mm_Horizontal, F.Cu at (118.5, 118.7)
- added R1: 100k, Resistor_THT:R_Axial_DIN0207_L6.3mm_D2.5mm_P7.62mm_Horizontal, F.Cu at (139.7, 109.6)
- added R3: 100k, Resistor_THT:R_Axial_DIN0207_L6.3mm_D2.5mm_P7.62mm_Horizontal, F.Cu at (134.9, 101.0)
- added R5: 10k, Resistor_THT:R_Axial_DIN0207_L6.3mm_D2.5mm_P7.62mm_Horizontal, F.Cu at (123.7, 111.2)
- added R6: 1k, Resistor_THT:R_Axial_DIN0204_L3.6mm_D1.6mm_P7.62mm_Horizontal, F.Cu at (147.2, 101.1)
- added U1: LTC1050, SHIELD_print_Library:LTC1050, F.Cu at (124.0, 99.9)
- added U2: Bluetooth-HC05, SHIELD_print_Library:HC-05, F.Cu at (134.5, 84.6)
- added U3: OLED_0.91, SHIELD_print_Library:SIP-4, F.Cu at (165.2, 106.1)
- added U4: Keyes_KY-040, SHIELD_print_Library:KY-040, F.Cu at (166.5, 86.4)
- added U5: MPC41100, SHIELD_print_Library:MPC41100_FP, F.Cu at (154.2, 87.6)
Connections:
- net /A4(SDA) renamed SDA
- net /A5(SCL) renamed SCL
- net /CMD-LED-D3 renamed /9(**)
- P2 pad 1: /A0 -> ADC
- P3 pad 10: /CMD-LED-D4 -> SCK
- P3 pad 5: /13(SCK) -> unconnected-(P3-Pad5)
- P3 pad 7: /CMD-LED-D1 -> TX
- P3 pad 8: /CMD-LED-D2 -> RX
- P4 pad 2: /6(**) -> SI
- P4 pad 3: /5(**) -> CS_
- P4 pad 4: /4 -> CLK
- P4 pad 5: /3(**) -> DATA
- P4 pad 6: /2 -> SWITCH
- P4 pad 7: /1(Tx) -> unconnected-(P4-Pad7)
- P4 pad 8: /0(Rx) -> unconnected-(P4-Pad8)
Routing:
- net +5V: track 0.00 -> 157.1 mm
- net IN-: track 0.00 -> 49.7 mm
- net IN+: track 0.00 -> 27.2 mm
- net Net-(C4-Pad1): track 0.00 -> 26.7 mm
- net ADC: track 0.00 -> 25.7 mm
- net SCL: track 0.00 -> 21.2 mm
- net SCK: track 0.00 -> 20.8 mm
- net PW0: track 0.00 -> 19.4 mm
- net SDA: track 0.00 -> 16.7 mm
- net RX: track 0.00 -> 15.8 mm
- net TX: track 0.00 -> 15.4 mm
- net SWITCH: track 0.00 -> 13.7 mm
- net DATA: track 0.00 -> 11.0 mm
- net SI: track 0.00 -> 10.9 mm
- net CS_: track 0.00 -> 9.84 mm
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