File: 2022-SHIELD-Arduino-FlexSensor/2022-SHIELD-Arduino-FlexSensor.kicad_sch (KiCad schematic)
At the start: 22 parts, among them P1 Power, P2 Analog, P3 Digital, P4 Digital, P5 CONN_01X01, P6 CONN_01X01, P7 CONN_01X01, P8 CONN_01X01, U1 LTC1050, U2 Bluetooth-HC05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

Commit message: Add files via upload
Parts:
- removed R2: 1k, symbol Device:R
- added U5: MPC41100, SHIELD_print_Library:MPC41100_FP, symbol SHIELD_Library:MPC41100
- C1, C3: footprint (none) -> Capacitor_THT:C_Disc_D4.3mm_W1.9mm_P5.00mm
- C2: footprint (none) -> Capacitor_THT:C_Disc_D7.5mm_W5.0mm_P7.50mm
- C4: footprint (none) -> Capacitor_THT:C_Rect_L7.0mm_W4.5mm_P5.00mm
- R1, R3, R5: footprint (none) -> Resistor_THT:R_Axial_DIN0207_L6.3mm_D2.5mm_P7.62mm_Horizontal
- R6: footprint (none) -> Resistor_THT:R_Axial_DIN0204_L3.6mm_D1.6mm_P7.62mm_Horizontal
Connections:
- net +5V: now also U5.8 (VDD)
- net GND: now also U5.4 (Vss), U5.5 (PA0), U5.6 (PWO)
- net IN-: now also U5.7 (PB0)
- net 0(Rx): no longer names the net of P4.8 (Pin_8)
- net 1(Tx): no longer names the net of P4.7 (Pin_7)
- net 13(SCK): no longer names the net of P3.5 (Pin_5)
- net 5(**) renamed CS_
- net CS_: now also U5.1 (CS_)
- net 6(**) renamed SI
- net SI: now also U5.3 (SI)
- net 8 renamed SCK
- net SCK: now also U5.2 (SCK)
- no-connect marks 29 -> 26
